File: PCB/PCB.sch (KiCad schematic (older format))
At the start: 4 parts

Commit message: Added PCB design files and wiring diagram
Parts:
- gave numbers to parts that had none: 4
Connections:
- net at U1.~ (GND), U3.~ (LV4): now also U2.~ (VCC)
- net at U3.~ (LV4): now also U4.~ (VCC); no longer U1.~ (GND)
- new net: U1.~ (GND), U3.~ (LV4) (x2)
- new net: U1.~ (GND), U2.~ (VCC), U3.~ (LV4)
- new net: U3.~ (LV4), U4.~ (VCC) (x2)
- no-connect marks 23 -> 25
Changed lines of the file:
@@
 $EndDescr
 $Comp
-L Adafruit:GrandCentralM4 U?
+L Adafruit:GrandCentralM4 U1
 U 1 1 5E11890F
 P 3350 4000
-F 0 "U?" H 3350 4000 50  0001 C CNN
+F 0 "U1" H 3350 4000 50  0001 C CNN
 F 1 "GrandCentralM4" H 3367 4573 50  0000 C CNN
 F 2 "" H 3300 3950 50  0001 C CNN
@@
 	6700 4150 6700 4050
 $Comp
-L OpenXPBMS:LogicConverter U?
+L OpenXPBMS:LogicConverter U3
 U 1 1 5E122D03
 P 5300 4050
-F 0 "U?" H 5300 4525 50  0001 C CNN
+F 0 "U3" H 5300 4525 50  0001 C CNN
 F 1 "LogicConverter" H 5300 4433 50  0000 C CNN
 F 2 "" H 5200 4000 50  0001 C CNN
@@
 NoConn ~ 4350 3900
 $Comp
-L OpenXPBMS:RS485 U?
+L OpenXPBMS:RS485 U4
 U 1 1 5E12E709
 P 7100 4100
-F 0 "U?" H 7100 4475 50  0001 C CNN
+F 0 "U4" H 7100 4475 50  0001 C CNN
 F 1 "RS485" H 7100 4383 50  0000 C CNN
 F 2 "" H 7150 3800 50  0001 C CNN
@@
 NoConn ~ 5800 4200
 Wire Wire Line
-	4850 4400 2900 4400
+	4850 4400 4050 4400
 Wire Wire Line
 	2900 4400 2900 4200
@@
 AMP_CONNECTOR
 $Comp
-L OpenXPBMS:RelayBoard U?
+L OpenXPBMS:RelayBoard U2
 U 1 1 5E141414
 P 3550 5050
-F 0 "U?" H 3608 5475 50  0001 C CNN
+F 0 "U2" H 3608 5475 50  0001 C CNN
 F 1 "RelayBoard" H 3608 5383 50  0000 C CNN
 F 2 "" H 3600 5050 50  0001 C CNN
@@
 Wire Wire Line
 	3800 3900 4450 3900
+Wire Wire Line
+	3800 5350 4050 5350
+Wire Wire Line
+	4050 5350 4050 4400
+Connection ~ 4050 4400
+Wire Wire Line
+	4050 4400 2900 4400
+NoConn ~ 4050 4450
+NoConn ~ 4050 4500
 $EndSCHEMATC
